Commit message: Fix cooked simulation logic, improve line follower tracking stability and optimize traffic light visibility

File: src/robo_description/urdf/robo404.gazebo.xacro (robot description, xacro)
@@ -62,5 +62,6 @@
       <visualize>true</visualize>
       <camera name="bottom_camera">
-        <horizontal_fov>1.0472</horizontal_fov>  <!-- 60 deg -->
+        <horizontal_fov>1.5708</horizontal_fov>  <!-- 90 deg: wider view so the
+             line stays in frame through the U-turns -->
         <image>
           <width>640</width>
@@ -91,5 +92,5 @@
       <visualize>true</visualize>
       <camera name="top_camera">
-        <horizontal_fov>1.0472</horizontal_fov>  <!-- 60 deg -->
+        <horizontal_fov>1.3962634</horizontal_fov>  <!-- 80 deg -->
         <image>
           <width>640</width>

File: src/robo_description/urdf/robo404.urdf.xacro (robot description, xacro)
@@ -28,5 +28,5 @@
   <xacro:property name="bot_cam_x" value="${chassis_length/2 - 0.01}" />
   <xacro:property name="bot_cam_z" value="0.06"  />
-  <xacro:property name="bot_cam_pitch" value="0.35" />   <!-- ~20 deg down -->
+  <xacro:property name="bot_cam_pitch" value="0.52" />   <!-- ~30 deg down -->
   <!-- top camera placement (looks forward/slightly up for traffic lights) -->
   <xacro:property name="top_cam_x" value="0.0" />
